Commit message: Changes for affnet and noetic

File: urdf/tiago159_with_zed.urdf.xacro (robot description, xacro)
@@ -27,4 +27,5 @@
     <xacro:arg name="extrinsic_calibration_dir" default="$(find tiago_dual_description_calibration)/urdf/calibration"/>
     <xacro:arg name="namespace" default=""/>
+    <xacro:arg name="fixed_torso" default="false" />
     <xacro:arg name="no_safety_eps" default="false"/>
     <xacro:property name="wrist_left_model" value="$(arg wrist_left_model)" />
@@ -45,4 +46,5 @@
     <xacro:property name="nsp" value="$(arg namespace)" />
     <xacro:property name="no_safety_eps" value="$(arg no_safety_eps)" />
+    <xacro:property name="fixed_torso" value="$(arg fixed_torso)" />
   <xacro:if value="${wrist_left_model not in ['wrist-2010', 'wrist-2017']}">
     <xacro:wrong_wrist_model/>
